File: heli-servo-board.kicad_pcb (KiCad board)
At the start: 2 copper layers, 20 x 24 mm, 13 parts, among them J1 Conn_01x06, J2 Conn_01x03, J3 Conn_01x03, J4 Conn_01x03, J6 Conn_01x02, J7 Conn_01x01, J8 Conn_01x01, J9 Conn_01x01

Commit message: Overdo the traces.
Routing:
- net Net-(J1-Pad3): track 16.0 -> 20.9 mm
- net Net-(J1-Pad1): track 5.73 -> 9.29 mm
- net Net-(J1-Pad2): track 11.2 -> 14.6 mm
Changed lines of the file:
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@@
     (thickness 1.6)
     (drawings 30)
-    (tracks 22)
+    (tracks 43)
     (zones 0)
     (modules 13)
@@
     (effects (font (size 0.8 0.8) (thickness 0.153)))
   )
-  (gr_text - (at 163.195 161.417) (layer F.SilkS)
-    (effects (font (size 0.8 0.8) (thickness 0.153)))
-  )
-  (gr_text + (at 163.195 160.147) (layer F.SilkS)
-    (effects (font (size 0.8 0.8) (thickness 0.153)))
-  )
-  (gr_text 1 (at 163.195 158.877) (layer F.SilkS)
+  (gr_text - (at 161.925 161.417) (layer F.SilkS)
+    (effects (font (size 0.8 0.8) (thickness 0.153)))
+  )
+  (gr_text + (at 161.925 160.147) (layer F.SilkS)
+    (effects (font (size 0.8 0.8) (thickness 0.153)))
+  )
+  (gr_text 1 (at 161.925 158.877) (layer F.SilkS)
     (effects (font (size 0.8 0.8) (thickness 0.153)))
   )
   (segment (start 173.792 152.877) (end 173.322 152.877) (width 0.6) (layer F.Cu) (net 1))
-  (segment (start 175.895 154.98) (end 173.792 152.877) (width 0.6) (layer F.Cu) (net 1))
   (segment (start 170.434 156.464) (end 168.824194 156.464) (width 0.6) (layer F.Cu) (net 1) (status 1000000))
   (segment (start 168.824194 156.464) (end 166.371194 158.917) (width 0.6) (layer F.Cu) (net 1) (status 1000000))
@@
   (segment (start 171.021982 155.921956) (end 170.976044 155.921956) (width 0.6) (layer F.Cu) (net 1) (status 1000000))
   (segment (start 170.976044 155.921956) (end 170.434 156.464) (width 0.6) (layer F.Cu) (net 1) (status 1000000))
-  (segment (start 171.021982 154.177018) (end 171.021982 155.921956) (width 0.6) (layer F.Cu) (net 1) (status 1000000))
-  (segment (start 172.322 152.877) (end 171.021982 154.177018) (width 0.6) (layer F.Cu) (net 1) (status 1000000))
   (segment (start 173.322 152.877) (end 172.322 152.877) (width 0.6) (layer F.Cu) (net 1) (status 1000000))
+  (segment (start 171.851 153.436) (end 171.807 153.392) (width 0.6) (layer F.Cu) (net 1))
+  (segment (start 171.807 153.392) (end 171.021982 154.177018) (width 0.6) (layer F.Cu) (net 1))
+  (segment (start 172.322 152.877) (end 171.807 153.392) (width 0.6) (layer F.Cu) (net 1))
+  (segment (start 175.895 154.98) (end 174.351 153.436) (width 0.6) (layer F.Cu) (net 1))
+  (segment (start 174.351 153.436) (end 173.792 152.877) (width 0.6) (layer F.Cu) (net 1))
+  (segment (start 172.446 153.436) (end 171.021982 154.860018) (width 0.6) (layer F.Cu) (net 1))
+  (segment (start 172.827 153.436) (end 172.446 153.436) (width 0.6) (layer F.Cu) (net 1))
+  (segment (start 171.021982 154.860018) (end 171.021982 155.921956) (width 0.6) (layer F.Cu) (net 1))
+  (segment (start 171.021982 154.177018) (end 171.021982 154.860018) (width 0.6) (layer F.Cu) (net 1))
+  (segment (start 174.351 153.436) (end 172.827 153.436) (width 0.6) (layer F.Cu) (net 1))
+  (segment (start 172.827 153.436) (end 171.851 153.436) (width 0.6) (layer F.Cu) (net 1))
   (segment (start 173.477678 154.909) (end 173.322 154.909) (width 0.6) (layer F.Cu) (net 2))
-  (segment (start 174.798678 156.23) (end 173.477678 154.909) (width 0.6) (layer F.Cu) (net 2))
   (segment (start 175.895 156.23) (end 174.798678 156.23) (width 0.6) (layer F.Cu) (net 2))
   (segment (start 169.927194 158.917) (end 167.894 158.917) (width 0.6) (layer F.Cu) (net 2) (status 1000000))
   (segment (start 173.322 154.909) (end 172.322 154.909) (width 0.6) (layer F.Cu) (net 2) (status 1000000))
-  (segment (start 171.82199 155.40901) (end 171.82199 157.022204) (width 0.6) (layer F.Cu) (net 2) (status 1000000))
   (segment (start 172.322 154.909) (end 171.82199 155.40901) (width 0.6) (layer F.Cu) (net 2) (status 1000000))
   (segment (start 171.82199 157.022204) (end 169.927194 158.917) (width 0.6) (layer F.Cu) (net 2) (status 1000000))
+  (segment (start 171.911141 155.498161) (end 171.82199 155.40901) (width 0.6) (layer F.Cu) (net 2))
+  (segment (start 174.798678 156.23) (end 174.066839 155.498161) (width 0.6) (layer F.Cu) (net 2))
+  (segment (start 174.066839 155.498161) (end 173.477678 154.909) (width 0.6) (layer F.Cu) (net 2))
+  (segment (start 172.542839 155.498161) (end 171.82199 156.21901) (width 0.6) (layer F.Cu) (net 2))
+  (segment (start 172.643161 155.498161) (end 172.542839 155.498161) (width 0.6) (layer F.Cu) (net 2))
+  (segment (start 171.82199 156.21901) (end 171.82199 157.022204) (width 0.6) (layer F.Cu) (net 2))
+  (segment (start 171.82199 155.40901) (end 171.82199 156.21901) (width 0.6) (layer F.Cu) (net 2))
+  (segment (start 174.066839 155.498161) (end 172.643161 155.498161) (width 0.6) (layer F.Cu) (net 2))
+  (segment (start 172.643161 155.498161) (end 171.911141 155.498161) (width 0.6) (layer F.Cu) (net 2))
   (segment (start 173.988 157.48) (end 173.322 156.814) (width 0.6) (layer F.Cu) (net 3))
-  (segment (start 175.895 157.48) (end 173.988 157.48) (width 0.6) (layer F.Cu) (net 3))
-  (segment (start 173.322 157.045) (end 171.45 158.917) (width 0.6) (layer F.Cu) (net 3) (status 1000000))
   (segment (start 173.322 156.814) (end 173.322 157.045) (width 0.6) (layer F.Cu) (net 3) (status 1000000))
+  (segment (start 172.887 157.48) (end 172.867 157.5) (width 0.6) (layer F.Cu) (net 3))
+  (segment (start 174.371 157.48) (end 172.887 157.48) (width 0.6) (layer F.Cu) (net 3))
+  (segment (start 175.895 157.48) (end 174.371 157.48) (width 0.6) (layer F.Cu) (net 3))
+  (segment (start 172.867 157.5) (end 171.45 158.917) (width 0.6) (layer F.Cu) (net 3))
+  (segment (start 173.322 157.045) (end 172.867 157.5) (width 0.6) (layer F.Cu) (net 3))
+  (segment (start 174.371 157.48) (end 173.988 157.48) (width 0.6) (layer F.Cu) (net 3))
+  (segment (start 171.45 158.525578) (end 172.621998 157.35358) (width 0.6) (layer F.Cu) (net 3))
+  (segment (start 171.45 158.917) (end 171.45 158.525578) (width 0.6) (layer F.Cu) (net 3))
   (zone (net 5) (net_name +BATT) (layer F.Cu) (hatch edge 0.508)
     (connect_pads yes (clearance 0.508))

Commit message: Fix Y dimension.
Parts:
- moved H1 4.00 mm to (160.0, 146.0)
- moved H3 4.00 mm to (176.0, 146.0)
Other:
- board size 20 x 24 mm -> 20 x 20 mm
